File: chassis/chassis.sch (KiCad schematic (older format))
At the start: 82 parts, among them J1 RJ45_LED_Shielded, Q1 FDG1024NZ, Q2 MMDT3906, T1 Transformer_1P_2S, T2 Transformer_1P_1S, U1 S558-5500-25-F, U2 TPS23754PWPR, U3 TCMT1107, U4 L78L33_SO8, U5 KSZ8081RND, U6 EFM32GG11B8xx

Commit message: hardware/*: various fixes based on review
Parts:
- removed C1, C16: 10n, Capacitor_SMD:C_0402_1005Metric, symbol Device:C
- removed D1, D6: D_Zener, Diode_SMD:D_0402_1005Metric, symbol Device:D_Zener
- removed Q1: FDG1024NZ, Package_TO_SOT_SMD:SOT-363_SC-70-6, symbol Transistor_FET:FDG1024NZ
- removed R11: ?, Resistor_SMD:R_0402_1005Metric, symbol Device:R
- removed R15: 1K, Resistor_SMD:R_0402_1005Metric, symbol Device:R
- removed R7: 130K, Resistor_SMD:R_0402_1005Metric, symbol Device:R
- removed R8: 15K, Resistor_SMD:R_0402_1005Metric, symbol Device:R
- removed T1: Transformer_1P_2S, symbol Device:Transformer_1P_2S
- removed T2: Transformer_1P_1S, symbol Device:Transformer_1P_1S
- removed U1: S558-5500-25-F, chassis:SOIC-16, symbol chassis:S558-5500-25-F
- removed U2: TPS23754PWPR, chassis:TSSOP-20, symbol chassis:TPS23754PWPR
- added C23: 330p, Capacitor_SMD:C_0402_1005Metric, symbol Device:C
- added C25: 1n, Capacitor_SMD:C_0402_1005Metric, symbol Device:C
- added FB1, FB2: Ferrite_Bead_Small, Resistor_SMD:R_1206_3216Metric, symbol Device:Ferrite_Bead_Small
- added Q1: SiR422DP, Package_SO:PowerPAK_SO-8_Single, symbol chassis:SiR422DP
- added Q2: Si7898DP, Package_SO:PowerPAK_SO-8_Single, symbol chassis:Si7898DP
- added R19: 1k, Resistor_SMD:R_0402_1005Metric, symbol Device:R
- added R20: 115k, Resistor_SMD:R_0402_1005Metric, symbol Device:R
- added R21: 560, Resistor_SMD:R_0402_1005Metric, symbol Device:R
- added R22: 13k3, Resistor_SMD:R_0402_1005Metric, symbol Device:R
- added T1: PoE_Transformer, chassis:POE_EP13, symbol chassis:PoE_Transformer
- added T2: Pulse_Transformer, chassis:GDTI_EP7, symbol chassis:Pulse_Transformer
- added TR1: PT61017PEL, Transformer_SMD:Transformer_Ethernet_Bourns_PT61017PEL, symbol Transformer:PT61017PEL
- added U1: TPS23754PWPR, Package_SO:HTSSOP-20-1EP_4.4x6.5mm_P0.65mm_EP3.4x6.5mm, symbol chassis:TPS23754PWPR
- added U3: TCMT1107, Package_SO:SOP-4_4.4x2.6mm_P1.27mm, symbol Isolator:TCMT1107
- C1: renamed from C3; Voltage (none) -> 100V
- C10: renamed from C2; value 1u2 -> 1n2
- C12: renamed from C13; Voltage (none) -> 25V
- C13: renamed from C14; Voltage (none) -> 100V
- C14: renamed from C15; Voltage (none) -> 100V
- C15: renamed from C17; Voltage (none) -> 2kV
- C18: renamed from C20; Voltage (none) -> 100V
- C19: renamed from C21; Voltage (none) -> 100V
- C2: renamed from C4; Voltage (none) -> 63V
- C20: renamed from C22; Voltage (none) -> 100V
- C21: renamed from C23; Voltage (none) -> 100V
- C3: renamed from C5; Voltage (none) -> 100V
- C4: renamed from C6; Voltage (none) -> 100V
- C5: renamed from C7; Voltage (none) -> 100V
- D1: renamed from D2; Voltage (none) -> 200V
- D3: renamed from D4; Voltage (none) -> 100V
- L2: value 3u3 -> 0u33
- R1, R4: value 68 -> 82
- R12: renamed from R16; Wattage (none) -> 0.5W
- R13: renamed from R18; value 10K -> 10k
- R14: renamed from R17; value 2K -> 2k
- R2: renamed from R3; Wattage (none) -> 0.25W
- R23: value 1K -> 1k
- R24: value 6K49 -> 6k49
- R5: value 24K9 -> 24k9
- R7: renamed from R9; value 38K3 -> 22k1
- R8: renamed from R10; value 69K8 -> 69k8
- R9: renamed from R12; value 69K8 -> 69k8
- U2: renamed from U3; footprint Package_SO:SOP-4_4.4x2.8mm_P1.27mm -> Package_SO:SOP-4_4.4x2.6mm_P1.27mm
- renumbered C12 to C11, C18 to C16, C19 to C17, C24 to C22, C25 to C24, C28 to C26, C29 to C27, C30 to C28, C31 to C29, C32 to C30, C33 to C31, C34 to C32, C35 to C33, C26 to C34, C27 to C35, C8 to C6, C9 to C7, C10 to C8, C11 to C9, D3 to D2, D7 to D4, D8 to D5, D5 to D6, Q2 to Q3, R13 to R10, R14 to R11, R19 to R15, R20 to R16, R21 to R17, R22 to R18, R2 to R3, U5 to U4, U4 to U5
Connections:
- net labels added: ETH_LED, GNDD, T2P, VC
- net labels removed: ETH_LED_ACT, GND
- wire segments 368 -> 373
Other:
- note added: "Class 4"
- note added: "Classification Resistor\n\nClass 0 (0.44 W-13W) - 1270 Ohm\nClass 1 (0.44 W-3.84 W) - 243 Ohm\nClass 2 (3.84 W-6.49 W) - 137 Ohm\nClass 3 (6.49 W-13 W) - 90.9 Ohm\nClass 4 (13 W-25.5 W) - 63.4 Ohm"
- moved on the sheet: C10, C11, C12, C15, C16, C17, C22, C24, C34, C35, C6, C7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

Commit message: hardware/lib: use new RJ-45 jack
Parts:
- J1: footprint chassis:RJMG1BD3B8K1ANR -> chassis:RJHSE-538X
Changed lines of the file:
@@
 F 0 "J1" H 2100 2167 50  0000 C CNN
 F 1 "RJ45_LED_Shielded" H 2100 2076 50  0000 C CNN
-F 2 "chassis:RJMG1BD3B8K1ANR" V 2100 1525 50  0001 C CNN
+F 2 "chassis:RJHSE-538X" V 2100 1525 50  0001 C CNN
 F 3 "~" V 2100 1525 50  0001 C CNN
 	1    2100 1500

Commit message: hardware/*: finalize initial schematic and layout
This marks the initial revision of the board.
Parts:
- removed R21: 560, Resistor_SMD:R_0402_1005Metric, symbol Device:R
- added 12V1, GND1: TestPoint, TestPoint:TestPoint_Loop_D1.80mm_Drill1.0mm_Beaded, symbol Connector:TestPoint
- added 3V3, GND2, PD0, PD1, PD2, PD3, PD4, PD5, PD6, PD8, PE4, PE5, PE6, PE7, PF10, PF11, TP? (x4), VDDA1, VSSA1: TestPoint, TestPoint:TestPoint_Pad_1.5x1.5mm, symbol Connector:TestPoint
- added R22: 100, Resistor_SMD:R_0402_1005Metric, symbol Device:R
- R1, R4: value 82 -> 1k2
- renumbered R14 to R13, R13 to R14, R22 to R21
Connections:
- net +12V: now also 12V1.1
- net +3V3: now also 3V3.1, R22.1; no longer R1.2, R4.2
- net CTL: now also TP?.1
- net ETH_LED: now also U3.1; no longer U4.23 (LED0/ANEN_SPEED)
- net ETH_RX_C: now also TR1.2 (C_TD); no longer TR1.7 (C_RD)
- net ETH_TX_C: now also TR1.7 (C_RD); no longer TR1.2 (C_TD)
- net GNDD: now also GND1.1, GND2.1; no longer U3.2
- net T2P: now also J1.11; no longer U3.3
- net VC: now also R1.2, R4.2
- net VDDA: now also VDDA1.1
- net VSSA: now also U3.2, VSSA1.1; no longer U1.10 (VSS), U1.21 (EPAD)
- net at U6.28 (PD0): now also PD0.1
- net at U6.29 (PD1): now also PD1.1
- net at U6.30 (PD2): now also PD2.1
- net at U6.31 (PD3): now also PD3.1
- net at U6.32 (PD4): now also PD4.1
- net at U6.33 (PD5): now also PD5.1
- net at U6.34 (PD6): now also PD6.1
- net at U6.35 (PD8): now also PD8.1
- net at U6.41 (PE4): now also PE4.1
- net at U6.42 (PE5): now also PE5.1
- net at U6.43 (PE6): now also PE6.1
- net at U6.44 (PE7): now also PE7.1
- net at U6.47 (PF10): now also PF10.1
- net at U6.48 (PF11): now also PF11.1
- net RX+: now reaches TR1.16 (TX+)
- net RX+: now also J1.3; no longer J1.1
- net RX-: now reaches TR1.14 (TX-)
- net RX-: now also J1.6; no longer J1.2
- net TX-: now reaches TR1.11 (RX+)
- net TX-: now also J1.2; no longer J1.3
- net TX+: now reaches TR1.9 (RX-)
- net TX+: now also J1.1; no longer J1.6
- net at C14.2, D3.2 (A), FB2.1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: now also U1.10 (VSS), U1.21 (EPAD)
- net at D5.3 (~~), TR1.10 (C_RX): now also C21.1; no longer C20.1
- net at D5.4 (~~), TR1.15 (C_TX): now also C20.1; no longer C21.1
- net at Q2.4 (G), R10.1: now also TP?.1
- net at C22.1, T2.3 (AB): now also TP?.1
- net at Q1.4 (G), Q3.1 (E1): now also TP?.1
- net at U3.4: now also R22.2
- net ETH_RX_M renamed ETH_RX-
- net ETH_RX_P renamed ETH_RX+
- net ETH_TX_M renamed ETH_TX-
- net ETH_TX_P renamed ETH_TX+
- removed net POE_LED: J1.11, U3.1
- new net ETH_LED0: U3.3, U4.23 (LED0/ANEN_SPEED)
- no-connect marks 46 -> 32
Other:
- note added: "REVERSE POLARITY OF THIS SIDE"
- moved on the sheet: C24, D6, R13, R19, R20, R21, U2

Commit message: chassis: various fixes
Parts:
- D3: Voltage 100V -> 58V
- gave numbers to parts that had none: 4
Changed lines of the file:
@@
 F 2 "Diode_SMD:D_0402_1005Metric" H 6000 2150 50  0001 C CNN
 F 3 "~" H 6000 2150 50  0001 C CNN
-F 4 "100V" V 6100 2300 50  0000 C CNN "Voltage"
+F 4 "58V" V 6100 2300 50  0000 C CNN "Voltage"
 	1    6000 2150
 	0    1    1    0
@@
 $EndComp
 $Comp
-L Connector:TestPoint TP?
+L Connector:TestPoint TP4
 U 1 1 5E1B7989
 P 14700 3300
-F 0 "TP?" H 14800 3550 50  0000 R CNN
+F 0 "TP4" H 14800 3550 50  0000 R CNN
 F 1 "TestPoint" V 14745 3488 50  0001 L CNN
 F 2 "TestPoint:TestPoint_Pad_1.5x1.5mm" H 14900 3300 50  0001 C CNN
@@
 	14700 3300 14900 3300
 $Comp
-L Connector:TestPoint TP?
+L Connector:TestPoint TP1
 U 1 1 5E1B9E90
 P 13500 2300
-F 0 "TP?" H 13600 2550 50  0000 R CNN
+F 0 "TP1" H 13600 2550 50  0000 R CNN
 F 1 "TestPoint" V 13545 2488 50  0001 L CNN
 F 2 "TestPoint:TestPoint_Pad_1.5x1.5mm" H 13700 2300 50  0001 C CNN
@@
 Connection ~ 13550 2300
 $Comp
-L Connector:TestPoint TP?
+L Connector:TestPoint TP3
 U 1 1 5E1E8923
 P 10150 3300
-F 0 "TP?" H 10250 3550 50  0000 R CNN
+F 0 "TP3" H 10250 3550 50  0000 R CNN
 F 1 "TestPoint" V 10195 3488 50  0001 L CNN
 F 2 "TestPoint:TestPoint_Pad_1.5x1.5mm" H 10350 3300 50  0001 C CNN
@@
 	10150 3300 9700 3300
 $Comp
-L Connector:TestPoint TP?
+L Connector:TestPoint TP2
 U 1 1 5E1EBBC9
 P 11250 2600
-F 0 "TP?" H 11350 2850 50  0000 R CNN
+F 0 "TP2" H 11350 2850 50  0000 R CNN
 F 1 "TestPoint" V 11295 2788 50  0001 L CNN
 F 2 "TestPoint:TestPoint_Pad_1.5x1.5mm" H 11450 2600 50  0001 C CNN
