File: hardware/sync-flyback-eval/sync-flyback-eval.kicad_sch (KiCad schematic)
At the start: 89 parts, among them J1 RJ45_LED_Shielded, Q1 SiR422DP, Q2 Si7898DP, Q3 MMDT3906, T1 PoE_Transformer, T2 Pulse_Transformer, U1 TPS23754PWPR, U2 TCMT1107

Commit message: flyback: specify range of trimpots
Parts:
- R7, R8, R9: value R_Trim -> 0-200k
Changed lines of the file:
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@@
     (in_bom yes) (on_board yes)
     (property "Reference" "R7" (id 0) (at 52.07 55.88 90))
-    (property "Value" "R_Trim" (id 1) (at 57.15 52.07 90)
+    (property "Value" "0-200k" (id 1) (at 57.15 52.07 90)
       (effects (font (size 1.27 1.27)) hide)
     )
@@
     (in_bom yes) (on_board yes)
     (property "Reference" "R9" (id 0) (at 52.07 60.96 90))
-    (property "Value" "R_Trim" (id 1) (at 57.15 57.15 90)
+    (property "Value" "0-200k" (id 1) (at 57.15 57.15 90)
       (effects (font (size 1.27 1.27)) hide)
     )
@@
     (in_bom yes) (on_board yes)
     (property "Reference" "R8" (id 0) (at 52.07 58.42 90))
-    (property "Value" "R_Trim" (id 1) (at 57.15 54.61 90)
+    (property "Value" "0-200k" (id 1) (at 57.15 54.61 90)
       (effects (font (size 1.27 1.27)) hide)
     )
@@
     )
     (path "/02e378bb-a850-4b7f-8f17-6b13b375af50"
-      (reference "R7") (unit 1) (value "R_Trim") (footprint "")
+      (reference "R7") (unit 1) (value "0-200k") (footprint "")
     )
     (path "/5a2c61f0-c5fd-40b6-b9e5-647b7568be4c"
-      (reference "R8") (unit 1) (value "R_Trim") (footprint "")
+      (reference "R8") (unit 1) (value "0-200k") (footprint "")
     )
     (path "/129986a3-7352-47a6-b6c6-91da1164e5f6"
-      (reference "R9") (unit 1) (value "R_Trim") (footprint "")
+      (reference "R9") (unit 1) (value "0-200k") (footprint "")
     )
     (path "/00000000-0000-0000-0000-00005c50e979"
