File: hardware/passthru/passthru.kicad_pcb (KiCad board)
At the start: 2 copper layers, 63.5 x 59.7 mm, 83 parts, among them J1 ARM_SWD, J2 RJ45_LED_Shielded, J3 Screw_Terminal_01x02, Q1 Q_PMOS_DGS, Q2 Q_PMOS_DGS, Q3 Q_NPN_BEC, U1 EFM32GG11B8xx, U2 KSZ8081RND, U3 LM5085, U4 TPS2375-1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

Commit message: passthru: cleanup silkscreen
Removed the part designators from the one side of the board, since they
really aren't necessary, and removed the redundant "+" from the
caution label.
Other:
- board text added: "Caution 57 V DC"
- board text added: "Caution: 57 V DC"
- board text removed: "Caution +57 V DC"
- board text removed: "Caution: +57 V DC"
Changed lines of the file:
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@@
     (property "Sheetname" "")
     (attr through_hole)
-    (fp_text reference "J3" (at -9.271 -10.414) (layer "B.SilkS")
+    (fp_text reference "J3" (at -9.271 -10.414) (layer "B.SilkS") hide
       (effects (font (size 0.75 0.75) (thickness 0.15)) (justify mirror))
     )
@@
     (property "Sheetname" "")
     (attr through_hole)
-    (fp_text reference "D2" (at 1.27 3.46) (layer "B.SilkS")
+    (fp_text reference "D2" (at 1.27 3.46) (layer "B.SilkS") hide
       (effects (font (size 0.75 0.75) (thickness 0.15)) (justify mirror))
     )
@@
     (property "Sheetname" "")
     (attr through_hole)
-    (fp_text reference "J2" (at 0 12.7) (layer "B.SilkS")
+    (fp_text reference "J2" (at 0 -3.746) (layer "B.SilkS") hide
       (effects (font (size 0.75 0.75) (thickness 0.15)) (justify mirror))
     )
@@
     (property "Sheetname" "")
     (attr through_hole)
-    (fp_text reference "D1" (at 1.27 3.46) (layer "B.SilkS")
+    (fp_text reference "D1" (at 1.27 3.46) (layer "B.SilkS") hide
       (effects (font (size 0.75 0.75) (thickness 0.15)) (justify mirror))
     )
@@
   (gr_arc (start 177.8 117.475) (mid 176.684077 120.169077) (end 173.99 121.285) (layer "Edge.Cuts") (width 0.1))
   (gr_arc (start 118.11 121.285) (mid 115.415923 120.169077) (end 114.3 117.475) (layer "Edge.Cuts") (width 0.1))
-  (gr_text "Identify" (at 162.56 99.06) (layer "B.SilkS")
+  (gr_text "Identify" (at 163.195 99.06) (layer "B.SilkS")
     (effects (font (size 1.5 1.5) (thickness 0.3)) (justify right mirror))
   )
-  (gr_text "Caution  +57 V DC" (at 123.19 90.805 180) (layer "B.SilkS")
+  (gr_text "Caution  57 V DC" (at 123.19 90.805 180) (layer "B.SilkS")
     (effects (font (size 1 1) (thickness 0.2)) (justify mirror))
   )
-  (gr_text "Caution: +57 V DC" (at 123.825 72.009) (layer "B.SilkS")
+  (gr_text "Caution: 57 V DC" (at 123.825 72.009) (layer "B.SilkS")
     (effects (font (size 1 1) (thickness 0.2)) (justify mirror))
   )
@@
     (effects (font (size 1.5 1.5) (thickness 0.3)) (justify right mirror))
   )
-  (gr_text "Caution: +57 V DC" (at 134.239 81.28 270) (layer "B.SilkS")
+  (gr_text "Caution: 57 V DC" (at 134.239 81.28 270) (layer "B.SilkS")
     (effects (font (size 1 1) (thickness 0.2)) (justify mirror))
   )

Commit message: passthru: replace network error led with general one
Rename the "Network" LED to "Error". Now that the firmware supports
occulting codes, this will be used for general error reporting. I also
included a preliminary error code chart. I hope this doesn't prove to
be too limiting.
Other:
- board text added: "Error"
- board text added: "No config (DHCP)"
- board text added: "No gateway (Router)"
- board text added: "No link (Ethernet)"
- board text removed: "Network"
Changed lines of the file:
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@@
     )
   )
+  (gr_circle (center 171.45 77.47) (end 171.7675 76.835) (layer "B.SilkS") (width 0.15) (fill none))
+  (gr_circle (center 171.45 80.01) (end 171.7675 79.375) (layer "B.SilkS") (width 0.15) (fill none))
+  (gr_rect (start 144.78 75.565) (end 173.355 84.455) (layer "B.SilkS") (width 0.15) (fill none))
+  (gr_circle (center 169.545 80.01) (end 169.8625 79.375) (layer "B.SilkS") (width 0.15) (fill none))
+  (gr_circle (center 171.45 82.55) (end 171.1325 81.915) (layer "B.SilkS") (width 0.15) (fill none))
+  (gr_circle (center 167.64 82.55) (end 167.3225 81.915) (layer "B.SilkS") (width 0.15) (fill none))
+  (gr_circle (center 169.545 82.55) (end 169.2275 81.915) (layer "B.SilkS") (width 0.15) (fill none))
   (gr_poly
     (pts
@@
   (gr_arc (start 177.8 117.475) (mid 176.684077 120.169077) (end 173.99 121.285) (layer "Edge.Cuts") (width 0.1))
   (gr_arc (start 118.11 121.285) (mid 115.415923 120.169077) (end 114.3 117.475) (layer "Edge.Cuts") (width 0.1))
+  (gr_text "No config (DHCP)" (at 164.465 80.01) (layer "B.SilkS")
+    (effects (font (size 1.2 1.2) (thickness 0.3)) (justify left mirror))
+  )
   (gr_text "Identify" (at 163.195 99.06) (layer "B.SilkS")
     (effects (font (size 1.5 1.5) (thickness 0.3)) (justify right mirror))
@@
     (effects (font (size 1 1) (thickness 0.2)) (justify mirror))
   )
+  (gr_text "No link (Ethernet)" (at 164.465 77.47) (layer "B.SilkS")
+    (effects (font (size 1.2 1.2) (thickness 0.3)) (justify left mirror))
+  )
   (gr_text "Caution: 57 V DC" (at 123.825 72.009) (layer "B.SilkS")
     (effects (font (size 1 1) (thickness 0.2)) (justify mirror))
   )
-  (gr_text "Network" (at 162.56 91.44) (layer "B.SilkS")
+  (gr_text "No gateway (Router)" (at 164.465 82.55) (layer "B.SilkS")
+    (effects (font (size 1.2 1.2) (thickness 0.3)) (justify left mirror))
+  )
+  (gr_text "Error" (at 163.195 91.44) (layer "B.SilkS")
     (effects (font (size 1.5 1.5) (thickness 0.3)) (justify right mirror))
   )
